Commit message: Adding state-based navigation and fixing bouncing

File: ros2_ws/src/micromouse_description/urdf/gazebo_control.xacro (robot description, xacro)
@@ -7,5 +7,5 @@
             <right_joint>right_wheel_joint</right_joint>
             <wheel_separation>0.35</wheel_separation>
-            <wheel_radius>0.05</wheel_radius>
+            <wheel_diameter>0.1</wheel_diameter>
             <!-- Limits -->
             <max_wheel_torque>200.0</max_wheel_torque>

File: ros2_ws/src/micromouse_description/urdf/mouse_core.xacro (robot description, xacro)
@@ -5,17 +5,17 @@
         <color rgba="1 1 1 1" />
     </material>
-    <material name="gray1">
-        <color rgba="0.5 0.5 0.5 1" />
+    <material name="orange">
+        <color rgba="1 0.3 0.1 1"/>
     </material>
-    <material name="gray2">
-        <color rgba="0.7 0.7 0.7 1" />
+    <material name="blue">
+        <color rgba="0.2 0.2 1 1"/>
     </material>
     <material name="black">
         <color rgba="0 0 0 1"/>
     </material>
-    <!--  Base link -->
+    <!-- BASE LINK -->
     <link name="base_link">
     </link>
-    <!-- Chassis Link -->
+    <!-- CHASSIS LINK -->
     <joint name="chassis_joint" type="fixed">
         <parent link="base_link"/>
@@ -44,5 +44,5 @@
         <material>Gazebo/White</material>
     </gazebo>
-    <!-- Left Wheel Link -->
+    <!-- LEFT WHEEL LINK -->
     <joint name="left_wheel_joint" type="continuous">
         <parent link="base_link"/>
@@ -56,5 +56,5 @@
                 <cylinder radius="0.05" length="0.04"/>
             </geometry>
-            <material name="gray1"/>
+            <material name="blue"/>
         </visual>
         <collision>
@@ -68,7 +68,7 @@
     </link>
     <gazebo reference="left_wheel">
-        <material>Gazebo/Black</material>
+        <material>Gazebo/Blue</material>
     </gazebo>
-    <!-- Right Wheel Link -->
+    <!-- RIGHT WHEEL LINK -->
     <joint name="right_wheel_joint" type="continuous">
         <parent link="base_link"/>
@@ -82,5 +82,5 @@
                 <cylinder radius="0.05" length="0.04"/>
             </geometry>
-            <material name="gray1"/>
+            <material name="blue"/>
         </visual>
         <collision>
@@ -94,7 +94,7 @@
     </link>
     <gazebo reference="right_wheel">
-        <material>Gazebo/Black</material>
+        <material>Gazebo/Blue</material>
     </gazebo>
-    <!-- Caster Wheel Link -->
+    <!-- CASTER WHEEL LINK -->
     <joint name="caster_wheel_joint" type="fixed">
         <parent link="chassis"/>
@@ -120,8 +120,7 @@
     <gazebo reference="caster_wheel">
         <material>Gazebo/Black</material>
-        <mul value="0.01"/>
-        <mu2 value="0.01"/>
+        <mu1 value="0.001"/>
+        <mu2 value="0.001"/>
     </gazebo>
-    <!-- Addomg pdp,etru tp Gazenp -->
     <gazebo>
         <plugin name="diff_drive_controller" filename="libgazebo_ros_diff_drive.so">
