Commit message: Fixed initial drift and increased turn precision at the cost of speed for development purposes

File: ros2_ws/src/micromouse_description/urdf/lidar.xacro (robot description, xacro)
@@ -31,8 +31,8 @@
                 <scan>
                     <horizontal>
-                        <samples>1</samples>
+                        <samples>4</samples>
                         <resolution>1</resolution>
-                        <min_angle>0</min_angle> <!-- -45 degrees -->
-                        <max_angle>0</max_angle> <!-- 45 degrees -->
+                        <min_angle>0</min_angle>
+                        <max_angle>4.71239</max_angle>
                     </horizontal>
                 </scan>

File: ros2_ws/src/micromouse_description/urdf/mouse_core.xacro (robot description, xacro)
@@ -16,4 +16,9 @@
     <!-- BASE LINK -->
     <link name="base_link">
+        <inertial>
+            <mass value="1.0"/>
+            <origin xyz="0 0 0" rpy="0 0 0"/>
+            <inertia ixx="0.1" ixy="0.0" ixz="0.0" iyy="0.1" iyz="0.0" izz="0.1"/>
+        </inertial>
     </link>
     <!-- CHASSIS LINK -->

Commit message: Implemented wall following navigation (admittedly at a slow pace

File: ros2_ws/src/micromouse_description/urdf/lidar.xacro (robot description, xacro)
@@ -38,6 +38,6 @@
                 </scan>
                 <range>
-                    <min>0.3</min>
-                    <max>20</max>
+                    <min>0.1</min>
+                    <max>1</max>
                     <resolution>0.01</resolution>
                 </range>

File: ros2_ws/src/micromouse_description/urdf/mouse_core.xacro (robot description, xacro)
@@ -65,6 +65,14 @@
         <collision>
             <geometry>
-                <cylinder radius="0.05" length="0.04"/>
+            <cylinder radius="0.05" length="0.04"/>
             </geometry>
+            <surface>
+            <friction>
+                <ode>
+                <mu>3.0</mu>
+                <mu2>3.0</mu2>
+                </ode>
+            </friction>
+            </surface>
         </collision>
         <xacro:inertial_cylinder mass="0.1" length="0.04" radius="0.05">
@@ -91,6 +99,14 @@
         <collision>
             <geometry>
-                <cylinder radius="0.05" length="0.04"/>
+            <cylinder radius="0.05" length="0.04"/>
             </geometry>
+            <surface>
+            <friction>
+                <ode>
+                <mu>3.0</mu>
+                <mu2>3.0</mu2>
+                </ode>
+            </friction>
+            </surface>
         </collision>
         <xacro:inertial_cylinder mass="0.1" length="0.04" radius="0.05">
